Commit message: Add files via upload

File: urdf/gingerurdf.urdf (robot description, URDF)
Before this commit: robot gingerurdf, 50 links, 49 joints
Joints:
- joint Left_Shoulder_X: origin xyz=0.167642819139667 -0.257434208387602 0.0153204612848375 rpy=1.5707963267949 0 -1.919840807 -> xyz=0.1634 -0.2581 0.0170 rpy=1.5707963267949 0 -1.919840807
- joint Right_Shoulder_X: origin xyz=-0.167642819137822 -0.257434208389716 0.0153204612848374 rpy=-1.5707963267949 0 -1.221709106 -> xyz=-0.1634 -0.2581 0.0170 rpy=-1.5707963267949 0 -1.221709106

Commit message: sssss

File: urdf/gingerurdf.urdf (robot description, URDF)
Before this commit: robot gingerurdf, 50 links, 49 joints
Joints:
- joint Left_Elbow_Z: origin xyz=0.0491247882 0.2246558260 0 rpy=0 1.5707963267949 1.5707963267949 -> xyz=0.049200 0.224520 0 rpy=0 1.5707963267949 1.5707963267949
- joint Left_Wrist_Z: origin xyz=0 0.209557803287771 0 rpy=-1.5707963267949 0 0 -> xyz=0 0.219230 0 rpy=-1.5707963267949 0 0
- joint Right_Elbow_Z: origin xyz=-0.0491247882 0.2246558260 0 rpy=0 1.5707963267949 1.5707963267949 -> xyz=-0.049200 0.224520 0 rpy=0 1.5707963267949 1.5707963267949
- joint Right_Wrist_Z: origin xyz=0 0.209559555159009 0 rpy=-1.5707963267949 0 0 -> xyz=0 0.219230 0 rpy=-1.5707963267949 0 0

Commit message: update armvalues

File: urdf/gingerurdf.urdf (robot description, URDF)
Before this commit: robot gingerurdf, 50 links, 49 joints
Joints:
- joint Left_Shoulder_X: origin xyz=0.1634 -0.2581 0.0170 rpy=1.5707963267949 0 -1.919840807 -> xyz=0.16340 -0.25810 0.01700 rpy=1.5707963267949 0 -1.919840807

Commit message: delete base link inertia

File: urdf/gingerurdf.urdf (robot description, URDF)
Before this commit: robot gingerurdf, 50 links, 49 joints
Links:
- link base_link: mass 36.8100641165154 -> None

Commit message: nothing

File: urdf/gingerurdf.urdf (robot description, URDF)
Before this commit: robot gingerurdf, 50 links, 49 joints
Links:
- link base_link: mass None -> 36.8100641165154

Commit message: merge safelimit branch
Change-Id: I75974b70ef12910bf4e6f0dccde67e5868611f69

File: urdf/gingerurdf.urdf (robot description, URDF)
Before this commit: robot gingerurdf, 50 links, 49 joints
Joints:
- removed joint Knee
- added joint Knee_X: type revolute, parent base_link, child Knee_Link, origin xyz=0 -0.163753578960292 0.422732937784996 rpy=1.5707963267949 0 1.5707963267949, axis 0 0 1, limit lower=-0.62779493194236 upper=0.539830337641846 effort=30 velocity=1.0
- joint Left_Elbow_X: limit lower=-1.61512768979555 upper=0.6770132168486 effort=30 velocity=1.0 -> lower=-2.100000 upper=0.6770132168486 effort=30 velocity=1.0
- joint Right_Elbow_X: limit lower=-1.61512768979555 upper=0.6770132168486 effort=30 velocity=1.0 -> lower=-2.100000 upper=0.6770132168486 effort=30 velocity=1.0

Commit message: add a joint Back_Y_Old

File: urdf/gingerurdf.urdf (robot description, URDF)
Before this commit: robot gingerurdf, 50 links, 49 joints
Links:
- added link Back_Y_Link_Old, mass 14.5524894817025; collision mesh filename=package://gingerurdf/meshes/Back_Y_Link.STL; visual mesh filename=package://gingerurdf/meshes/Back_Y_Link.STL
Joints:
- added joint Back_Y_Old: type revolute, parent Back_X_Link, child Back_Y_Link_Old, origin xyz=0.104999999999997 0 0 rpy=-1.5707963267949 0 0, axis 0 0 1, limit lower=-0.720820981073658 upper=0.720820981073658 effort=30 velocity=1.0
- joint Back_Y: origin xyz=0.104999999999997 0 0 rpy=0 -1.5707963267949 1.5707963267949 -> xyz=0 0 0 rpy=3.141592654 0 -1.5707963267949; parent Back_X_Link -> Back_Y_Link_Old

Commit message: delete backyold, change rshouldery range

File: urdf/gingerurdf.urdf (robot description, URDF)
Before this commit: robot gingerurdf, 51 links, 50 joints
Links:
- removed link Back_Y_Link_Old
Joints:
- removed joint Back_Y_Old
- joint Back_Y: origin xyz=0 0 0 rpy=3.141592654 0 -1.5707963267949 -> xyz=0.105 0 0 rpy=0 -1.5707963267949 1.5707963267949; parent Back_Y_Link_Old -> Back_X_Link
- joint Right_Shoulder_Y: limit lower=-1.73084301920278 upper=0.0162315620435473 effort=30 velocity=1.0 -> lower=-0.0162315620435473 upper=1.73084301920278 effort=30 velocity=1.0

Commit message: update joint range
Change-Id: Ic0c07e2f3e8d703985f7b6a78f7ed8107381c0bb

File: urdf/gingerurdf.urdf (robot description, URDF)
Before this commit: robot gingerurdf, 50 links, 49 joints
Joints:
- removed joint Knee
- added joint Knee_X: type revolute, parent base_link, child Knee_Link, origin xyz=0 -0.163753578960292 0.422732937784996 rpy=1.5707963267949 0.0562043157596906 -2.28428512229131, axis -0.653442120633779 -0.0367649880485583 -0.756083150609388, limit lower=-0.62779493194236 upper=0.539830337641846 effort=30 velocity=1.0
- joint Left_Elbow_X: limit lower=-1.61512768979555 upper=0.6770132168486 effort=30 velocity=1.0 -> lower=-2.13333 upper=0.6770132168486 effort=30 velocity=1.0
- joint Left_Wrist_Z: limit lower=-1.5707963267949 upper=1.5707963267949 effort=30 velocity=1.0 -> lower=-2.093333 upper=2.093333 effort=30 velocity=1.0
- joint Right_Elbow_X: limit lower=-1.61512768979555 upper=0.6770132168486 effort=30 velocity=1.0 -> lower=-2.1333 upper=0.6770132168486 effort=30 velocity=1.0
- joint Right_Wrist_Z: limit lower=-1.5707963267949 upper=1.5707963267949 effort=30 velocity=1.0 -> lower=-2.093333 upper=2.0933333 effort=30 velocity=1.0
